File: kicad/10k-Hour-Timer-RP2040.kicad_pcb (KiCad board)
At the start: 2 copper layers, 245 x 173 mm, 102 parts, among them J1 JST_SH_SM03B, J2 USB_C_Receptacle_USB2.0_16P, J3 S2B-PH-K-S_LF__SN_, Q1 PMOS, Q2 AO3400A, Q3 AO3400A, Q4 AO3400A, Q5 AO3400A, U1 USBLC6-2SC6, U2 MCP73831-2-OT, U3 BQ29700DSER, U4 TLV62568DBV, U5 W25Q128JVS, U6 PCF8523T, U7 RP2040, Y1 ABS07AIG-32.768KHZ-7-T, Y2 ABM8-272-T3

Commit message: DR SYS-02-DCDC ✅
Parts:
- added C6: 4.7u, Capacitor_SMD:C_0603_1608Metric_Pad1.08x0.95mm_HandSolder, F.Cu at (109.4, 41.0)
- added C8: 22u, Capacitor_SMD:C_0603_1608Metric_Pad1.08x0.95mm_HandSolder, F.Cu at (99.9, 35.5)
- added TP22: DC_SW, project footprints:TestPoint_THTPad_D2.0mm_Drill1.0mm, F.Cu at (126.5, 29.0)
- TP15: value TestPoint -> EN_CTL
- U4: value TLV62568DBV -> TLV62568DBVR
- moved JP8 160.2 mm to (99.7, 39.8)
- moved JP7 155.9 mm to (104.4, 39.2)
- moved TP15 146.5 mm to (120.8, 29.0)
- moved R13 141.8 mm to (114.5, 27.8)
- moved R14 141.4 mm to (114.5, 31.5)
- moved R15 141.4 mm to (114.5, 34.5)
- moved R16 141.4 mm to (114.5, 37.4)
- moved D6 135.1 mm to (121.4, 37.0)
- moved U4 102.8 mm to (108.4, 30.0)
- moved C9 90.0 mm to (104.4, 35.5)
- moved C7 76.8 mm to (108.9, 35.2)
- moved L1 70.9 mm to (102.0, 29.8)
- moved U1 25.1 mm to (154.0, 80.0)
- moved J1 25.1 mm to (95.3, 85.3)
- moved Y1 25.1 mm to (149.7, 88.3)
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Connections:
- net Net-(JP8-A) renamed /01-04-Power-DCDC-Charger-Battery/DC_EN_CTL
- net Net-(U4-FB) renamed /01-04-Power-DCDC-Charger-Battery/DC_FB
Other:
- board text added: "DCDC"
