File: kicad/10k-Hour-Timer-RP2040.kicad_pcb (KiCad board)
At the start: 2 copper layers, 245 x 173 mm, 143 parts, among them J1 JST_SH_SM03B, J2 USB_C_Receptacle_USB2.0_16P, J3 S2B-PH-K-S_LF__SN_, J6 Conn_01x03_Pin, J7 Conn_01x03_Pin, J8 Conn_01x03_Pin, J9 Conn_01x12_Pin, Q1 PMOS, Q2 AO3400A, Q3 AO3400A, Q4 AO3400A, Q5 AO3400A, SW1 BOOTSEL, SW2 RESET, SW3 USER_A, SW4 USER_B_PWR, U1 USBLC6-2SC6, U2 MCP73831-2-OT, U3 BQ29700DSER, U4 TLV62568DBVR, U5 W25Q128JVS, U6 PCF8523T, U7 RP2040, Y1 ABS07AIG-32.768KHZ-7-T, Y2 ABM8-272-T3

Commit message: pre ERC
Parts:
- removed the JP19 at (256.6, 125.5)
- removed the R23 at (241.5, 54.5)
- removed the R25 at (241.5, 60.5)
- removed the R40 at (300.8, 51.2)
- removed the U6 at (128.5, 123.2)
- removed the Y1 at (152.7, 112.0)
- added BT1: Battery_Cell, project footprints:Battery-Holder-BH-123A_37.5P_1.8D_MH, F.Cu at (142.2, 111.8)
- added C1: 0.1u, Capacitor_SMD:C_0805_2012Metric_Pad1.18x1.45mm_HandSolder, F.Cu at (-21.8, 154.1)
- added C2: 4u7, Capacitor_SMD:C_0805_2012Metric_Pad1.18x1.45mm_HandSolder, F.Cu at (-21.8, 157.1)
- added C23: 2.2u, Capacitor_SMD:C_0805_2012Metric_Pad1.18x1.45mm_HandSolder, F.Cu at (192.0, 78.3)
- added C24: 100n, Capacitor_SMD:C_0805_2012Metric_Pad1.18x1.45mm_HandSolder, F.Cu at (192.0, 81.3)
- added C25: 4.7u, Capacitor_SMD:C_0805_2012Metric_Pad1.18x1.45mm_HandSolder, F.Cu at (179.7, 79.7)
- added D10: RED/INT, LED_SMD:LED_0805_2012Metric, F.Cu at (184.6, 76.4)
- added J10: S2B-PH-K-S_LF__SN_, Connector_JST:JST_PH_S2B-PH-K_1x02_P2.00mm_Horizontal, F.Cu at (114.9, 44.0)
- added J11: Conn_01x02_Pin, Connector_PinHeader_2.54mm:PinHeader_1x02_P2.54mm_Vertical, F.Cu at (122.2, 43.9)
- added J5: Conn_02x05_Counter_Clockwise, Connector_PinHeader_2.54mm:PinHeader_2x05_P2.54mm_Vertical, F.Cu at (314.2, 136.6)
- added J9: Conn_01x02_Pin, Connector_PinHeader_2.54mm:PinHeader_1x02_P2.54mm_Vertical, F.Cu at (323.3, 136.6)
- added JP21: SolderJumper_2_Open, Jumper:SolderJumper-2_P1.3mm_Open_RoundedPad1.0x1.5mm, F.Cu at (171.1, 83.2)
- added JP23: SolderJumper_2_Open, Jumper:SolderJumper-2_P1.3mm_Open_RoundedPad1.0x1.5mm, F.Cu at (171.1, 86.7)
- added Q6: PMOS, Package_TO_SOT_SMD:SOT-23, F.Cu at (184.5, 83.8)
- added R20: 10K, Resistor_SMD:R_0805_2012Metric_Pad1.20x1.40mm_HandSolder, F.Cu at (316.5, 86.4)
- added R21: 10K, Resistor_SMD:R_0805_2012Metric_Pad1.20x1.40mm_HandSolder, F.Cu at (316.5, 83.4)
- added R22: 10K, Resistor_SMD:R_0805_2012Metric_Pad1.20x1.40mm_HandSolder, F.Cu at (316.5, 80.5)
- added R41: 1K, Resistor_SMD:R_0805_2012Metric_Pad1.20x1.40mm_HandSolder, F.Cu at (175.6, 82.9)
- added R42: 470, Resistor_SMD:R_0805_2012Metric_Pad1.20x1.40mm_HandSolder, F.Cu at (175.6, 85.8)
- added R43: 100K, Resistor_SMD:R_0805_2012Metric_Pad1.20x1.40mm_HandSolder, F.Cu at (175.6, 88.8)
- added SW6: SW_SPDT, Button_Switch_THT:SW_E-Switch_EG1271_SPDT, F.Cu at (170.2, 114.3)
- added TP24: INT_G, project footprints:TestPoint_THTPad_D2.0mm_Drill1.0mm, F.Cu at (180.0, 83.4)
- added TP25: INT_D, project footprints:TestPoint_THTPad_D2.0mm_Drill1.0mm, F.Cu at (180.0, 87.5)
- added TP26: LOAD, project footprints:TestPoint_THTPad_D2.0mm_Drill1.0mm, F.Cu at (121.9, 50.8)
- added U7: PCF8523T, Package_SO:SOIC-8_3.9x4.9mm_P1.27mm, F.Cu at (173.1, 78.2)
- added Y2: ABS07AIG-32.768KHZ-7-T, Crystal:Crystal_SMD_3215-2Pin_3.2x1.5mm, F.Cu at (179.9, 76.5)
- TP1: value TestPoint -> GND
- TP2: value TestPoint -> VBUS_IN
- TP3: value TestPoint -> VBUS
- TP4: value VBATT -> VBAT
- moved JP22 134.4 mm to (171.1, 90.3)
- renumbered BZ2 to BZ1, BZ1 to BZ2, C13 to C12, C14 to C13, C17 to C14, C18 to C15, C19 to C16, C20 to C17, C21 to C18, C22 to C19, C23 to C20, C24 to C21, C25 to C22, J8 to J1, J1 to J2, J2 to J3, J3 to J4, J9 to J6, J6 to J7, J7 to J8, JP20 to JP19, JP21 to JP20, R20 to R19, R22 to R23, R19 to R24, R21 to R25, R24 to R26, R26 to R27, R27 to R28, R28 to R29, R29 to R30, R30 to R31, R31 to R32, R32 to R33, R33 to R34, R34 to R35, R35 to R36, R36 to R37, R37 to R38, R38 to R39, R39 to R40, SW1 to SW2, SW2 to SW3, SW3 to SW4, SW4 to SW5, U7 to U6, Y2 to Y1
Connections:
- net /01-04-Power-DCDC-Charger-Battery/5V_USB renamed /Power-DCDC-Charger-Battery/5V_USB
- net /01-04-Power-DCDC-Charger-Battery/ADC1_VSW_In renamed /Power-DCDC-Charger-Battery/ADC1_VSW_In
- net /01-04-Power-DCDC-Charger-Battery/BTN_PWR renamed /Power-DCDC-Charger-Battery/BTN_PWR_RTC
- net /01-04-Power-DCDC-Charger-Battery/Batt- renamed /Power-DCDC-Charger-Battery/Batt-
- net /01-04-Power-DCDC-Charger-Battery/DC_EN_CTL renamed /Power-DCDC-Charger-Battery/DC_EN_CTL
- net /01-04-Power-DCDC-Charger-Battery/DC_FB renamed /Power-DCDC-Charger-Battery/DC_FB
- net /01-04-Power-DCDC-Charger-Battery/PWR_CTL renamed /Power-DCDC-Charger-Battery/PWR_CTL
- net /01-04-Power-DCDC-Charger-Battery/STAT renamed /Power-DCDC-Charger-Battery/STAT
- net /01-04-Power-DCDC-Charger-Battery/Vbatt renamed /Power-DCDC-Charger-Battery/Vbat
- net /05-07_MCU-LED-Driver-Displays/ADC0 renamed /MCU-IO/ADC0
- net /05-07_MCU-LED-Driver-Displays/ADC0_VUSB_In renamed /MCU-IO/ADC0_VUSB_In
- net /05-07_MCU-LED-Driver-Displays/ADC1 renamed /MCU-IO/ADC1
- net /05-07_MCU-LED-Driver-Displays/ADC1_VSW_In renamed /MCU-IO/ADC1_VSW_In
- net /05-07_MCU-LED-Driver-Displays/ADC2 renamed /MCU-IO/ADC2
- net /05-07_MCU-LED-Driver-Displays/ADC3 renamed /MCU-IO/ADC3
- net /05-07_MCU-LED-Driver-Displays/AVDD renamed /MCU-IO/AVDD
- net /05-07_MCU-LED-Driver-Displays/BTN_A_Sense renamed /MCU-IO/BTN_A_Sense
- net /05-07_MCU-LED-Driver-Displays/BTN_B_Sense renamed /MCU-IO/BTN_B_Sense
- net /05-07_MCU-LED-Driver-Displays/BZ1 renamed /MCU-IO/BZ1
- net /05-07_MCU-LED-Driver-Displays/BZ2_N renamed /MCU-IO/BZ2_N
- net /05-07_MCU-LED-Driver-Displays/BZ2_P renamed /MCU-IO/BZ2_P
- net /05-07_MCU-LED-Driver-Displays/DCDC_EN renamed /MCU-IO/DCDC_EN
- net /05-07_MCU-LED-Driver-Displays/DISP_CLK renamed /MCU-IO/DISP_CLK
- net /05-07_MCU-LED-Driver-Displays/DISP_DIO renamed /MCU-IO/DISP_DIO
- net /05-07_MCU-LED-Driver-Displays/DISP_STB renamed /MCU-IO/DISP_STB
- net /05-07_MCU-LED-Driver-Displays/GPIO15 renamed /MCU-IO/GPIO15
- net /05-07_MCU-LED-Driver-Displays/GPIO16 renamed /MCU-IO/GPIO16
- net /05-07_MCU-LED-Driver-Displays/IO10 renamed /MCU-IO/IO10
- net /05-07_MCU-LED-Driver-Displays/IO14 renamed /MCU-IO/IO14
- net /05-07_MCU-LED-Driver-Displays/IO2 renamed /MCU-IO/IO2
- net /05-07_MCU-LED-Driver-Displays/IO21 renamed /MCU-IO/IO21
- net /05-07_MCU-LED-Driver-Displays/IO22 renamed /MCU-IO/IO22
- net /05-07_MCU-LED-Driver-Displays/IO25_LED renamed /MCU-IO/IO25_LED
- net /05-07_MCU-LED-Driver-Displays/IO3 renamed /MCU-IO/IO3
- net /05-07_MCU-LED-Driver-Displays/IO4 renamed /MCU-IO/IO4
- net /05-07_MCU-LED-Driver-Displays/IO5 renamed /MCU-IO/IO5
- net /05-07_MCU-LED-Driver-Displays/IO9 renamed /MCU-IO/IO9
- net /05-07_MCU-LED-Driver-Displays/IO_Gate renamed /MCU-IO/IO_Gate
- net /05-07_MCU-LED-Driver-Displays/QSPI_CLK renamed /MCU-IO/QSPI_CLK
- net /05-07_MCU-LED-Driver-Displays/QSPI_SD0 renamed /MCU-IO/QSPI_SD0
- net /05-07_MCU-LED-Driver-Displays/QSPI_SD1 renamed /MCU-IO/QSPI_SD1
- net /05-07_MCU-LED-Driver-Displays/QSPI_SD2 renamed /MCU-IO/QSPI_SD2
- net /05-07_MCU-LED-Driver-Displays/QSPI_SD3 renamed /MCU-IO/QSPI_SD3
- net /05-07_MCU-LED-Driver-Displays/QSPI_SS renamed /MCU-IO/QSPI_SS
- net /05-07_MCU-LED-Driver-Displays/UART0_Rx renamed /MCU-IO/UART0_Rx
- net /05-07_MCU-LED-Driver-Displays/UART0_Tx renamed /MCU-IO/UART0_Tx
- net /05-07_MCU-LED-Driver-Displays/XIN renamed /MCU-IO/XIN
- net /05-07_MCU-LED-Driver-Displays/XOUT renamed /MCU-IO/XOUT
- net /05-07_MCU-LED-Driver-Displays/~{Reset} renamed /MCU-IO/~{Reset}
- J4 pad 1: /01-04-Power-DCDC-Charger-Battery/Batt+ -> Net-(BT1-+)
- J6 pad 8: /05-07_MCU-LED-Driver-Displays/IO17 -> unconnected-(J6-Pin_8-Pad8)
- J6 pad 9: /05-07_MCU-LED-Driver-Displays/IO18 -> unconnected-(J6-Pin_9-Pad9)
- JP14 pad 1: /05-07_MCU-LED-Driver-Displays/VDD_Out -> /MCU-IO/VDD_Out
- JP15 pad 1: /05-07_MCU-LED-Driver-Displays/GND_Out -> /MCU-IO/GND_Out
- JP16 pad 1: /05-07_MCU-LED-Driver-Displays/STB_Out -> /MCU-IO/STB_Out
- JP17 pad 1: /05-07_MCU-LED-Driver-Displays/CLK_Out -> /MCU-IO/CLK_Out
- JP18 pad 1: /05-07_MCU-LED-Driver-Displays/DIO_Out -> /MCU-IO/DIO_Out
- JP22 pad 1: 3V3 -> /RTC/RTC_INT_GPIN0
- JP22 pad 2: Net-(JP22-B) -> /RTC/INT_G
- R10 pad 2: /01-04-Power-DCDC-Charger-Battery/Batt+ -> /Power-DCDC-Charger-Battery/Batt+
- R24 pad 1: /05-07_MCU-LED-Driver-Displays/I2C_SDA -> /MCU-IO/RTC_SCL
- R25 pad 1: /05-07_MCU-LED-Driver-Displays/I2C_SCL -> /MCU-IO/RTC_SDA
- R9 pad 2: /01-04-Power-DCDC-Charger-Battery/Batt+ -> /Power-DCDC-Charger-Battery/Batt+
- TP8 pad 1: /01-04-Power-DCDC-Charger-Battery/Batt+ -> /Power-DCDC-Charger-Battery/Batt+
- U6 pad 28: /05-07_MCU-LED-Driver-Displays/IO17 -> /MCU-IO/RTC_SCL
- U6 pad 29: /05-07_MCU-LED-Driver-Displays/IO18 -> /MCU-IO/RTC_SDA
- U6 pad 31: /05-07_MCU-LED-Driver-Displays/RTC_INT_GPIN0 -> /MCU-IO/RTC_INT_GPIN0
Other:
- board text added: "RTC"

Commit message: ERC done
Parts:
- C1: value 0.1u -> 10n; footprint Capacitor_SMD:C_0805_2012Metric_Pad1.18x1.45mm_HandSolder -> Capacitor_SMD:C_0603_1608Metric_Pad1.08x0.95mm_HandSolder
- C2: value 4u7 -> 100n; footprint Capacitor_SMD:C_0805_2012Metric_Pad1.18x1.45mm_HandSolder -> Capacitor_SMD:C_0603_1608Metric_Pad1.08x0.95mm_HandSolder
- J6: value Conn_01x12_Pin -> Conn_01x13_Pin; footprint Connector_PinHeader_2.54mm:PinHeader_1x12_P2.54mm_Vertical -> Connector_PinHeader_2.54mm:PinHeader_1x13_P2.54mm_Vertical
- TP19: value TestPoint -> DCDC_EN
- TP23: value TestPoint -> ADC0
- moved J6 117.2 mm to (35.6, 104.1)
- moved C2 83.6 mm to (42.0, 103.1)
Connections:
- net /Power-DCDC-Charger-Battery/Vbat renamed /Power-DCDC-Charger-Battery/VBAT
- C2 pad 1: /Power-DCDC-Charger-Battery/5V_USB -> /MCU-IO/ADC0_VUSB_In
- C3 pad 1: /Power-DCDC-Charger-Battery/5V_USB -> /MCU-IO/ADC0_VUSB_In
- D2 pad 2: /Power-DCDC-Charger-Battery/5V_USB -> /MCU-IO/ADC0_VUSB_In
- D3 pad 1: /Power-DCDC-Charger-Battery/ADC1_VSW_In -> /MCU-IO/ADC1_VSW_In
- D4 pad 1: /Power-DCDC-Charger-Battery/ADC1_VSW_In -> /MCU-IO/ADC1_VSW_In
- D7 pad 1: /Power-DCDC-Charger-Battery/BTN_PWR_RTC -> /MCU-IO/IO_Gate
- FB1 pad 2: /Power-DCDC-Charger-Battery/5V_USB -> /MCU-IO/ADC0_VUSB_In
- J2 pad MP: GND -> unconnected-(J2-MountPin-PadMP)
- J6 pad 10: /MCU-IO/IO21 -> /MCU-IO/IO16
- J6 pad 11: /MCU-IO/IO22 -> /MCU-IO/IO21
- J6 pad 12: GND -> /MCU-IO/IO22
- J6 pad 7: /MCU-IO/IO14 -> /MCU-IO/IO10
- J6 pad 8: unconnected-(J6-Pin_8-Pad8) -> /MCU-IO/IO14
- J6 pad 9: unconnected-(J6-Pin_9-Pad9) -> /MCU-IO/IO15
- JP22 pad 1: /RTC/RTC_INT_GPIN0 -> /MCU-IO/RTC_INT_GPIN0
- JP23 pad 2: /RTC/BTN_PWR_RTC -> /MCU-IO/IO_Gate
- JP3 pad 2: /Power-DCDC-Charger-Battery/5V_USB -> /MCU-IO/ADC0_VUSB_In
- JP4 pad 2: /Power-DCDC-Charger-Battery/5V_USB -> /MCU-IO/ADC0_VUSB_In
- JP5 pad 1: /Power-DCDC-Charger-Battery/5V_USB -> /MCU-IO/ADC0_VUSB_In
- JP6 pad 2: /Power-DCDC-Charger-Battery/ADC1_VSW_In -> /MCU-IO/ADC1_VSW_In
- JP8 pad 2: /Power-DCDC-Charger-Battery/5V_USB -> /MCU-IO/ADC0_VUSB_In
- Q1 pad 2: /Power-DCDC-Charger-Battery/5V_USB -> /MCU-IO/ADC0_VUSB_In
- Q1 pad 3: /Power-DCDC-Charger-Battery/ADC1_VSW_In -> /MCU-IO/ADC1_VSW_In
- R14 pad 2: /Power-DCDC-Charger-Battery/PWR_CTL -> /MCU-IO/DCDC_EN
- R24 pad 1: /MCU-IO/RTC_SCL -> /MCU-IO/I2C_SCL
- R25 pad 1: /MCU-IO/RTC_SDA -> /MCU-IO/I2C_SDA
- TP3 pad 1: /Power-DCDC-Charger-Battery/5V_USB -> /MCU-IO/ADC0_VUSB_In
- TP5 pad 1: /Power-DCDC-Charger-Battery/5V_USB -> /MCU-IO/ADC0_VUSB_In
- TP6 pad 1: /Power-DCDC-Charger-Battery/ADC1_VSW_In -> /MCU-IO/ADC1_VSW_In
- U2 pad 4: /Power-DCDC-Charger-Battery/5V_USB -> /MCU-IO/ADC0_VUSB_In
- U6 pad 18: /MCU-IO/GPIO15 -> /MCU-IO/IO15
- U6 pad 19: unconnected-(U6-TESTEN-Pad19) -> GND
- U6 pad 27: /MCU-IO/GPIO16 -> /MCU-IO/IO16
- U6 pad 28: /MCU-IO/RTC_SCL -> /MCU-IO/I2C_SCL
- U6 pad 29: /MCU-IO/RTC_SDA -> /MCU-IO/I2C_SDA
- U7 pad 5: /RTC/I2C_SDA -> /MCU-IO/I2C_SDA
- U7 pad 6: /RTC/I2C_SCL -> /MCU-IO/I2C_SCL
