File: kicad/10k-Hour-Timer-RP2040.kicad_sch (KiCad schematic)
At the start: 12 parts, among them J1 JST_SH_SM03B, J2 USB_C_Receptacle_USB2.0_16P, U1 USBLC6-2SC6

Commit message: DR  ✅ SYS-01-Power-Mux
Parts:
- JP1: footprint (none) -> Jumper:SolderJumper-2_P1.3mm_Open_RoundedPad1.0x1.5mm
- R1, R2: footprint (none) -> Resistor_SMD:R_0805_2012Metric_Pad1.20x1.40mm_HandSolder
- TP1: renamed from TP12; footprint (none) -> project footprints:TestPoint_THTPad_D2.0mm_Drill1.0mm
- TP2: renamed from TP11; footprint (none) -> project footprints:TestPoint_THTPad_D2.0mm_Drill1.0mm
- TP3: renamed from TP13; footprint (none) -> project footprints:TestPoint_THTPad_D2.0mm_Drill1.0mm
Changed lines of the file:
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@@
+			)
+		)
+		(property "Subsystem" ""
+			(at 52.07 123.19 0)
+			(effects
+				(font
+					(size 1.27 1.27)
+				)
+				(hide yes)
 			)
 		)
@@
 			)
 		)
-		(property "Footprint" ""
+		(property "Footprint" "Jumper:SolderJumper-2_P1.3mm_Open_RoundedPad1.0x1.5mm"
 			(at 54.61 95.25 0)
 			(effects
@@
 			)
 		)
+		(property "Subsystem" ""
+			(at 54.61 95.25 0)
+			(effects
+				(font
+					(size 1.27 1.27)
+				)
+				(hide yes)
+			)
+		)
 		(pin "1"
 		)
@@
 			)
 		)
+		(property "Subsystem" ""
+			(at 109.22 60.96 0)
+			(effects
+				(font
+					(size 1.27 1.27)
+				)
+				(hide yes)
+			)
+		)
 		(pin "2"
 		)
@@
 			)
 		)
-		(property "Footprint" ""
+		(property "Footprint" "Resistor_SMD:R_0805_2012Metric_Pad1.20x1.40mm_HandSolder"
 			(at 82.55 64.008 90)
 			(effects
@@
 			)
 		)
+		(property "Subsystem" ""
+			(at 82.55 62.23 90)
+			(effects
+				(font
+					(size 1.27 1.27)
+				)
+				(hide yes)
+			)
+		)
 		(pin "2"
 		)
@@
 		(on_board yes)
 		(dnp no)
-		(property "Reference" "TP13"
+		(property "Reference" "TP3"
 			(at 129.7589 52.07 0)
 			(effects
@@
 			)
 		)
-		(property "Footprint" ""
+		(property "Footprint" "project footprints:TestPoint_THTPad_D2.0mm_Drill1.0mm"
 			(at 136.6169 57.15 0)
 			(effects
@@
 			)
 		)
+		(property "Subsystem" ""
+			(at 131.5369 57.15 0)
+			(effects
+				(font
+					(size 1.27 1.27)
+				)
+				(hide yes)
+			)
+		)
 		(pin "1"
 		)
@@
 			(project "10k-Hour-Timer-RP2040"
 				(path "/9d26b66f-2a94-42e5-8460-016e0bf95186"
-					(reference "TP13")
+					(reference "TP3")
 					(unit 1)
 				)
@@
 		(on_board yes)
 		(dnp no)
-		(property "Reference" "TP12"
+		(property "Reference" "TP1"
 			(at 62.738 95.504 90)
 			(effects
@@
 			)
 		)
-		(property "Footprint" ""
+		(property "Footprint" "project footprints:TestPoint_THTPad_D2.0mm_Drill1.0mm"
 			(at 58.42 100.33 0)
 			(effects
@@
 			)
 		)
+		(property "Subsystem" ""
+			(at 58.42 95.25 90)
+			(effects
+				(font
+					(size 1.27 1.27)
+				)
+				(hide yes)
+			)
+		)
 		(pin "1"
 		)
@@
 			(project "10k-Hour-Timer-RP2040"
 				(path "/9d26b66f-2a94-42e5-8460-016e0bf95186"
-					(reference "TP12")
+					(reference "TP1")
 					(unit 1)
 				)
@@
 		(on_board yes)
 		(dnp no)
-		(property "Reference" "TP11"
+		(property "Reference" "TP2"
 			(at 88.392 52.07 0)
 			(effects
@@
 			)
 		)
-		(property "Footprint" ""
+		(property "Footprint" "project footprints:TestPoint_THTPad_D2.0mm_Drill1.0mm"
 			(at 95.25 57.15 0)
 			(effects
@@
 			)
 		)
+		(property "Subsystem" ""
+			(at 90.17 57.15 0)
+			(effects
+				(font
+					(size 1.27 1.27)
+				)
+				(hide yes)
+			)
+		)
 		(pin "1"
 		)
@@
 			(project "10k-Hour-Timer-RP2040"
 				(path "/9d26b66f-2a94-42e5-8460-016e0bf95186"
-					(reference "TP11")
+					(reference "TP2")
 					(unit 1)
 				)
@@
 			)
 		)
+		(property "Subsystem" ""
+			(at 119.38 57.15 90)
+			(effects
+				(font
+					(size 1.27 1.27)
+				)
+				(hide yes)
+			)
+		)
 		(pin "2"
 		)
@@
 			)
 		)
+		(property "Subsystem" ""
+			(at 58.42 72.39 0)
+			(effects
+				(font
+					(size 1.27 1.27)
+				)
+				(hide yes)
+			)
+		)
 		(pin "A9"
 		)
@@
 			)
 		)
-		(property "Footprint" ""
+		(property "Footprint" "Resistor_SMD:R_0805_2012Metric_Pad1.20x1.40mm_HandSolder"
 			(at 82.55 66.548 90)
 			(effects
@@
 			)
 		)
+		(property "Subsystem" ""
+			(at 82.55 64.77 90)
+			(effects
+				(font
+					(size 1.27 1.27)
+				)
+				(hide yes)
+			)
+		)
 		(pin "2"
 		)
@@
 			)
 		)
+		(property "Subsystem" ""
+			(at 102.87 73.66 0)
+			(effects
+				(font
+					(size 1.27 1.27)
+				)
+				(hide yes)
+			)
+		)
 		(pin "2"
 		)
@@
 			(at 125.73 60.96 0)
 			(effects
+				(font
+					(size 1.27 1.27)
+				)
+				(hide yes)
+			)
+		)
+		(property "Subsystem" ""
+			(at 125.73 60.96 0)
+			(effects

Commit message: DR SYS-02-DCDC ✅
Parts:
- JP1, TP1, TP2, TP3: MPN (none) -> (Embedded)
Changed lines of the file:
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@@
+			)
+		)
+		(property "MPN" "(Embedded)"
+			(at 54.61 95.25 0)
+			(effects
+				(font
+					(size 1.27 1.27)
+				)
+				(hide yes)
 			)
 		)
@@
 			)
 		)
+		(property "MPN" "(Embedded)"
+			(at 131.5369 57.15 0)
+			(effects
+				(font
+					(size 1.27 1.27)
+				)
+				(hide yes)
+			)
+		)
 		(pin "1"
 		)
@@
 			)
 		)
+		(property "MPN" "(Embedded)"
+			(at 58.42 95.25 90)
+			(effects
+				(font
+					(size 1.27 1.27)
+				)
+				(hide yes)
+			)
+		)
 		(pin "1"
 		)
@@
 			(at 90.17 57.15 0)
 			(effects
+				(font
+					(size 1.27 1.27)
+				)
+				(hide yes)
+			)
+		)
+		(property "MPN" "(Embedded)"
+			(at 90.17 57.15 0)
+			(effects

Commit message: DR SYS-04-Battery Protect ✅
Parts:
- R1, R2: MPN (none) -> (Generic)
Changed lines of the file:
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@@
+			)
+		)
+		(property "MPN" "(Generic)"
+			(at 82.55 62.23 90)
+			(effects
+				(font
+					(size 1.27 1.27)
+				)
+				(hide yes)
 			)
 		)
@@
 			(at 82.55 64.77 90)
 			(effects
+				(font
+					(size 1.27 1.27)
+				)
+				(hide yes)
+			)
+		)
+		(property "MPN" "(Generic)"
+			(at 82.55 64.77 90)
+			(effects

Commit message: DR SYS-05-MCU XTAL
Parts:
- added J8: Conn_01x03_Pin, Connector_PinHeader_2.54mm:PinHeader_1x03_P2.54mm_Vertical, symbol Connector:Conn_01x03_Pin
- J1: Subsystem (none) -> 05-MCU-XTAL-FLASH
Connections:
- net GND: now also J8.2 (Pin_2)
- net SWCLK: now also J8.1 (Pin_1)
- net SWDIO: now also J8.3 (Pin_3)
Changed lines of the file:
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@@
 	(text "For use with RasPi debugger"
 		(exclude_from_sim no)
-		(at 54.61 139.446 0)
+		(at 61.976 152.908 0)
 		(effects
 			(font
@@
 	(text "NB. Rx/Tx from the Target/MCU POV"
 		(exclude_from_sim no)
-		(at 54.864 141.732 0)
+		(at 62.23 155.194 0)
 		(effects
 			(font
@@
 	(wire
 		(pts
+			(xy 59.69 146.05) (xy 73.66 146.05)
+		)
+		(stroke
+			(width 0)
+			(type default)
+		)
+	)
+	(wire
+		(pts
 			(xy 134.62 72.39) (xy 127 72.39)
 		)
@@
 	(wire
 		(pts
+			(xy 59.69 143.51) (xy 53.34 143.51)
+		)
+		(stroke
+			(width 0)
+			(type default)
+		)
+	)
+	(wire
+		(pts
 			(xy 127 97.79) (xy 133.35 97.79)
 		)
@@
 	(wire
 		(pts
+			(xy 59.69 146.05) (xy 59.69 143.51)
+		)
+		(stroke
+			(width 0)
+			(type default)
+		)
+	)
+	(wire
+		(pts
 			(xy 63.5 125.73) (xy 57.15 125.73)
 		)
@@
 	(wire
 		(pts
+			(xy 53.34 140.97) (xy 57.15 140.97)
+		)
+		(stroke
+			(width 0)
+			(type default)
+		)
+	)
+	(wire
+		(pts
 			(xy 123.19 57.15) (xy 125.73 57.15)
 		)
@@
 		(pts
 			(xy 127 72.39) (xy 127 97.79)
+		)
+		(stroke
+			(width 0)
+			(type default)
+		)
+	)
+	(wire
+		(pts
+			(xy 53.34 138.43) (xy 74.93 138.43)
 		)
 		(stroke
@@
 		)
 	)
+	(label "SWDIO"
+		(at 73.66 146.05 180)
+		(effects
+			(font
+				(size 1.27 1.27)
+			)
+			(justify right bottom)
+		)
+	)
 	(label "USB_D-"
 		(at 107.95 73.66 0)
@@
 			)
 			(justify left bottom)
+		)
+	)
+	(label "SWCLK"
+		(at 74.93 138.43 180)
+		(effects
+			(font
+				(size 1.27 1.27)
+			)
+			(justify right bottom)
+		)
+	)
+	(symbol
+		(lib_id "power:GND")
+		(at 57.15 140.97 90)
+		(unit 1)
+		(exclude_from_sim no)
+		(in_bom yes)
+		(on_board yes)
+		(dnp no)
+		(property "Reference" "#PWR066"
+			(at 63.5 140.97 0)
+			(effects
+				(font
+					(size 1.27 1.27)
+				)
+				(hide yes)
+			)
+		)
+		(property "Value" "GND"
+			(at 60.96 140.9699 90)
+			(effects
+				(font
+					(size 1.27 1.27)
+				)
+				(justify right)
+			)
+		)
+		(property "Footprint" ""
+			(at 57.15 140.97 0)
+			(effects
+				(font
+					(size 1.27 1.27)
+				)
+				(hide yes)
+			)
+		)
+		(property "Datasheet" ""
+			(at 57.15 140.97 0)
+			(effects
+				(font
+					(size 1.27 1.27)
+				)
+				(hide yes)
+			)
+		)
+		(property "Description" "Power symbol creates a global label with name \"GND\" , ground"
+			(at 57.15 140.97 0)
+			(effects
+				(font
+					(size 1.27 1.27)
+				)
+				(hide yes)
+			)
+		)
+		(pin "1"
+		)
+		(instances
+			(project "10k-Hour-Timer-RP2040"
+				(path "/9d26b66f-2a94-42e5-8460-016e0bf95186"
+					(reference "#PWR066")
+					(unit 1)
+				)
+			)
 		)
 	)
@@
 			)
 		)
-		(property "Subsystem" ""
+		(property "Subsystem" "05-MCU-XTAL-FLASH"
 			(at 52.07 123.19 0)
 			(effects
@@
 					(unit 1)
 				)
+			)
+		)
+	)
+	(symbol
+		(lib_id "Connector:Conn_01x03_Pin")
+		(at 48.26 140.97 0)
+		(unit 1)
+		(exclude_from_sim no)
+		(in_bom no)
+		(on_board yes)
+		(dnp no)
+		(property "Reference" "J8"
+			(at 46.99 139.6999 0)
+			(effects
+				(font
+					(size 1.27 1.27)
+				)
+				(justify right)
+			)
+		)
+		(property "Value" "Conn_01x03_Pin"
+			(at 46.99 142.2399 0)
+			(effects
+				(font
+					(size 1.27 1.27)
+				)
+				(justify right)
+			)
+		)
+		(property "Footprint" "Connector_PinHeader_2.54mm:PinHeader_1x03_P2.54mm_Vertical"
+			(at 48.26 140.97 0)
+			(effects
+				(font
+					(size 1.27 1.27)
+				)
+				(hide yes)
+			)
+		)
+		(property "Datasheet" "~"
+			(at 48.26 140.97 0)
+			(effects
+				(font
+					(size 1.27 1.27)
+				)
+				(hide yes)
+			)
+		)
+		(property "Description" "Generic connector, single row, 01x03, script generated"
+			(at 48.26 140.97 0)
+			(effects
+				(font
+					(size 1.27 1.27)
+				)
+				(hide yes)
+			)
+		)
+		(property "Subsystem" "05-MCU-XTAL-FLASH"
+			(at 48.26 140.97 0)
+			(effects
+				(font
+					(size 1.27 1.27)
+				)
+				(hide yes)
+			)
+		)
+		(property "MPN" "(Embedded)"
+			(at 48.26 140.97 0)
+			(effects
+				(font
+					(size 1.27 1.27)
+				)
+				(hide yes)
+			)
+		)
+		(property "Manufacturer" "(Embedded)"
+			(at 48.26 140.97 0)
+			(effects
+				(font
+					(size 1.27 1.27)
+				)
+				(hide yes)
+			)
+		)
+		(property "Supplier 1" "(Embedded)"
+			(at 48.26 140.97 0)
+			(effects
+				(font
+					(size 1.27 1.27)
+				)
+				(hide yes)
+			)
+		)
+		(pin "3"
+		)
+		(pin "2"
+		)
+		(pin "1"
+		)
+		(instances
+			(project ""
+				(path "/9d26b66f-2a94-42e5-8460-016e0bf95186"
+					(reference "J8")
+					(unit 1)
+				)

Commit message: DR SYS-06-MCU-IO ✅
Parts:
- FB1: Lab_In_Stock (none) -> Y
Other:
- note added: "typ. shield tied to ground on host side, leave device side floating"
- note removed: "typ shield tied to ground on host side, leave device side floating"
Changed lines of the file:
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@@
 		)
 	)
-	(text "typ shield tied to ground on host side, leave device side floating"
-		(exclude_from_sim no)
-		(at 56.388 105.156 0)
+	(text "typ. shield tied to ground on host side,\n leave device side floating"
+		(exclude_from_sim no)
+		(at 58.42 106.172 0)
 		(effects
 			(font
@@
 	(text "TODO - find Yokogawa compatible connectors for USB "
 		(exclude_from_sim no)
-		(at 60.96 45.974 0)
+		(at 58.166 36.83 0)
 		(effects
 			(font
@@
 	(wire
 		(pts
-			(xy 134.62 72.39) (xy 127 72.39)
+			(xy 144.78 72.39) (xy 137.16 72.39)
 		)
 		(stroke
@@
 	(wire
 		(pts
-			(xy 127 97.79) (xy 133.35 97.79)
+			(xy 137.16 111.76) (xy 143.51 111.76)
 		)
 		(stroke
@@
 	(wire
 		(pts
-			(xy 172.72 67.31) (xy 190.5 67.31)
+			(xy 182.88 67.31) (xy 190.5 67.31)
 		)
 		(stroke
@@
 	(wire
 		(pts
-			(xy 172.72 72.39) (xy 182.88 72.39)
-		)
-		(stroke
-			(width 0)
-			(type default)
-		)
-	)
-	(wire
-		(pts
 			(xy 63.5 128.27) (xy 77.47 128.27)
 		)
@@
 	(wire
 		(pts
-			(xy 111.76 118.11) (xy 133.35 118.11)
+			(xy 121.92 132.08) (xy 143.51 132.08)
 		)
 		(stroke
@@
 	(wire
 		(pts
-			(xy 172.72 62.23) (xy 191.77 62.23)
+			(xy 182.88 62.23) (xy 191.77 62.23)
 		)
 		(stroke
@@
 	(wire
 		(pts
-			(xy 111.76 113.03) (xy 133.35 113.03)
+			(xy 121.92 127) (xy 143.51 127)
 		)
 		(stroke
@@
 	(wire
 		(pts
-			(xy 119.38 102.87) (xy 133.35 102.87)
+			(xy 129.54 116.84) (xy 143.51 116.84)
 		)
 		(stroke
@@
 	(wire
 		(pts
-			(xy 127 72.39) (xy 127 97.79)
+			(xy 137.16 72.39) (xy 137.16 111.76)
 		)
 		(stroke
@@
 	(wire
 		(pts
-			(xy 119.38 107.95) (xy 133.35 107.95)
+			(xy 129.54 121.92) (xy 143.51 121.92)
 		)
 		(stroke
@@
 	(wire
 		(pts
-			(xy 172.72 57.15) (xy 186.69 57.15)
+			(xy 182.88 57.15) (xy 186.69 57.15)
 		)
 		(stroke
@@
 	(wire
 		(pts
-			(xy 131.5369 57.15) (xy 134.62 57.15)
+			(xy 131.5369 57.15) (xy 144.78 57.15)
 		)
 		(stroke
@@
 	)
 	(label "SWCLK"
-		(at 111.76 118.11 0)
+		(at 121.92 132.08 0)
 		(effects
 			(font
@@
 	)
 	(label "USB_D+"
-		(at 119.38 107.95 0)
+		(at 129.54 121.92 0)
 		(effects
 			(font
@@
 	)
 	(label "SWDIO"
-		(at 111.76 113.03 0)
+		(at 121.92 127 0)
 		(effects
 			(font
@@
 	)
 	(label "USB_D-"
-		(at 119.38 102.87 0)
+		(at 129.54 116.84 0)
 		(effects
 			(font
@@
 			)
 		)
+		(property "Lab_In_Stock" "Y"
+			(at 119.38 57.15 90)
+			(effects
+				(font
+					(size 1.27 1.27)
+				)
+				(hide yes)
+			)
+		)
 		(pin "2"
 		)
@@
 	)
 	(sheet
-		(at 133.35 93.98)
+		(at 143.51 107.95)
 		(size 38.1 31.75)
 		(exclude_from_sim no)
@@
 		)
 		(property "Sheetname" "05-07_MCU-LED-Driver-Displays"
-			(at 133.35 93.2684 0)
+			(at 143.51 107.2384 0)
 			(effects
 				(font
@@
 		)
 		(property "Sheetfile" "05-07_MCU-LED-Driver-Displays.kicad_sch"
-			(at 133.35 126.3146 0)
+			(at 143.51 140.2846 0)
 			(effects
 				(font
@@
 		)
 		(pin "USB_D+" input
-			(at 133.35 107.95 180)
+			(at 143.51 121.92 180)
 			(effects
 				(font
@@
 		)
 		(pin "USB_D-" input
-			(at 133.35 102.87 180)
+			(at 143.51 116.84 180)
 			(effects
 				(font
@@
 		)
 		(pin "SWD" input
-			(at 133.35 113.03 180)
+			(at 143.51 127 180)
 			(effects
 				(font
@@
 		)
 		(pin "SWCK" input
-			(at 133.35 118.11 180)
+			(at 143.51 132.08 180)
 			(effects
 				(font
@@
 		)
 		(pin "BTN_PWR" output
-			(at 171.45 99.06 0)
+			(at 181.61 113.03 0)
 			(effects
 				(font
@@
 		)
 		(pin "PWR_CTL" output
-			(at 171.45 104.14 0)
+			(at 181.61 118.11 0)
 			(effects
 				(font
@@
 		)
 		(pin "ADC0_VUSB_In" input
-			(at 171.45 109.22 0)
+			(at 181.61 123.19 0)
 			(effects
 				(font
@@
 		)
 		(pin "ADC1_VSW_In" input
-			(at 171.45 114.3 0)
+			(at 181.61 128.27 0)
 			(effects
 				(font
@@
 		)
 		(pin "Vbatt" input
-			(at 133.35 97.79 180)
+			(at 143.51 111.76 180)
 			(effects
 				(font
@@
 	)
 	(sheet
-		(at 134.62 52.07)
+		(at 144.78 52.07)
 		(size 38.1 26.67)
 		(exclude_from_sim no)
@@
 		)
 		(property "Sheetname" "01-04-Power-DCDC-Charger-Battery"
-			(at 134.62 51.3584 0)
+			(at 144.78 51.3584 0)
 			(effects
 				(font
@@
 		)
 		(property "Sheetfile" "01-04-Power-DCDC-Charger-Battery.kicad_sch"
-			(at 134.62 79.3246 0)
+			(at 144.78 79.3246 0)
 			(effects
 				(font
@@
 		)
 		(pin "5V_USB" input
-			(at 134.62 57.15 180)
+			(at 144.78 57.15 180)
 			(effects
 				(font
@@
 		)
 		(pin "BTN_PWR" input
-			(at 172.72 57.15 0)
+			(at 182.88 57.15 0)
 			(effects
 				(font
@@
 		)
 		(pin "PWR_CTL" input
-			(at 172.72 62.23 0)
+			(at 182.88 62.23 0)
 			(effects
 				(font
@@
 		)
 		(pin "ADC1_VSW_In" output
-			(at 172.72 72.39 0)
+			(at 182.88 72.39 0)
 			(effects
 				(font
@@
 		)
 		(pin "ADC0_VUSB_In" output
-			(at 172.72 67.31 0)
+			(at 182.88 67.31 0)
 			(effects
 				(font
@@
 		)
 		(pin "Vbatt" output
-			(at 134.62 72.39 180)
-			(effects
-				(font
+			(at 144.78 72.39 180)
+			(effects
+				(font
