File: kicad/01-04-Power-DCDC-Charger-Battery.kicad_sch (KiCad schematic)
At the start: 69 parts, among them J10 S2B-PH-K-S_LF__SN_, J11 Conn_01x02_Pin, J4 S2B-PH-K-S_LF__SN_, Q1 PMOS, Q2 AO3400A, Q3 AO3400A, SW6 SW_SPDT, U2 MCP73831-2-OT, U3 BQ29700DSER, U4 TLV62568DBVR

Commit message: layout floorplanning
Parts:
- removed JP8: SolderJumper_2_Bridged, Jumper:SolderJumper-2_P1.3mm_Bridged_RoundedPad1.0x1.5mm, symbol Jumper:SolderJumper_2_Bridged
- added TP5: U2_VDD, project footprints:TestPoint_THTPad_D2.0mm_Drill1.0mm, symbol Connector:TestPoint
- C3, C4: footprint Capacitor_SMD:C_0805_2012Metric_Pad1.18x1.45mm_HandSolder -> Capacitor_SMD:C_0603_1608Metric_Pad1.08x0.95mm_HandSolder; Package 0805 -> 0603
- C5: Package 0805 -> 0603
- C7: value 470n, 10V -> 470n
Connections:
- net 5V_USB: now also D6.2 (A), TP5.1
Changed lines of the file:
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@@
 	)
 	(junction
+		(at 162.56 34.29)
+		(diameter 0)
+		(color 0 0 0 0)
+	)
+	(junction
 		(at 52.07 134.62)
 		(diameter 0)
@@
 	(wire
 		(pts
+			(xy 162.56 34.29) (xy 166.37 34.29)
+		)
+		(stroke
+			(width 0)
+			(type default)
+		)
+	)
+	(wire
+		(pts
 			(xy 132.08 44.45) (xy 132.08 45.72)
 		)
@@
 	(wire
 		(pts
-			(xy 163.83 34.29) (xy 166.37 34.29)
-		)
-		(stroke
-			(width 0)
-			(type default)
-		)
-	)
-	(wire
-		(pts
 			(xy 96.52 152.4) (xy 96.52 149.86)
 		)
@@
 	(wire
 		(pts
-			(xy 143.51 34.29) (xy 156.21 34.29)
+			(xy 143.51 34.29) (xy 162.56 34.29)
 		)
 		(stroke
@@
 			)
 		)
-		(property "Footprint" "Capacitor_SMD:C_0805_2012Metric_Pad1.18x1.45mm_HandSolder"
+		(property "Footprint" "Capacitor_SMD:C_0603_1608Metric_Pad1.08x0.95mm_HandSolder"
 			(at 194.0052 38.1 0)
 			(effects
@@
 			)
 		)
-		(property "Package" "0805"
+		(property "Package" "0603"
 			(at 193.04 34.29 0)
 			(effects
@@
 			)
 		)
-		(property "Package" "0805"
+		(property "Package" "0603"
 			(at 52.07 143.51 0)
 			(effects
@@
 			)
 		)
-		(property "Footprint" "Capacitor_SMD:C_0805_2012Metric_Pad1.18x1.45mm_HandSolder"
+		(property "Footprint" "Capacitor_SMD:C_0603_1608Metric_Pad1.08x0.95mm_HandSolder"
 			(at 181.3052 38.1 0)
 			(effects
@@
 			)
 		)
-		(property "Package" "0805"
+		(property "Package" "0603"
 			(at 180.34 34.29 0)
 			(effects
@@
 			)
 		)
-		(property "Value" "470n, 10V"
+		(property "Value" "470n"
 			(at 168.91 131.826 0)
 			(effects
@@
 	)
 	(symbol
-		(lib_id "Jumper:SolderJumper_2_Bridged")
-		(at 160.02 34.29 180)
-		(unit 1)
-		(exclude_from_sim no)
-		(in_bom no)
-		(on_board yes)
-		(dnp no)
-		(property "Reference" "JP8"
-			(at 161.036 32.004 0)
-			(effects
-				(font
-					(size 1.27 1.27)
-				)
-				(justify right)
-			)
-		)
-		(property "Value" "SolderJumper_2_Bridged"
-			(at 161.2899 31.75 90)
-			(effects
-				(font
-					(size 1.27 1.27)
-				)
-				(justify right)
-				(hide yes)
-			)
-		)
-		(property "Footprint" "Jumper:SolderJumper-2_P1.3mm_Bridged_RoundedPad1.0x1.5mm"
-			(at 160.02 34.29 0)
-			(effects
-				(font
-					(size 1.27 1.27)
-				)
-				(hide yes)
-			)
-		)
-		(property "Datasheet" "~"
-			(at 160.02 34.29 0)
-			(effects
-				(font
-					(size 1.27 1.27)
-				)
-				(hide yes)
-			)
-		)
-		(property "Description" "Solder Jumper, 2-pole, closed/bridged"
-			(at 160.02 34.29 0)
-			(effects
-				(font
-					(size 1.27 1.27)
-				)
-				(hide yes)
-			)
-		)
-		(property "Subsystem" ""
-			(at 160.02 34.29 90)
-			(effects
-				(font
-					(size 1.27 1.27)
-				)
-				(hide yes)
-			)
-		)
-		(property "MPN" "(Embedded)"
-			(at 160.02 34.29 90)
-			(effects
-				(font
-					(size 1.27 1.27)
-				)
-				(hide yes)
-			)
-		)
-		(pin "2"
-		)
-		(pin "1"
-		)
-		(instances
-			(project "10k-Hour-Timer-RP2040"
-				(path "/9d26b66f-2a94-42e5-8460-016e0bf95186/9c84c2c8-9981-4486-adaf-4a40ca17b6d0"
-					(reference "JP8")
-					(unit 1)
-				)
-			)
-		)
-	)
-	(symbol
 		(lib_id "power:GND")
 		(at 132.08 53.34 0)
@@
 					(unit 1)
 				)
+			)
+		)
+	)
+	(symbol
+		(lib_id "Connector:TestPoint")
+		(at 162.56 34.29 0)
+		(unit 1)
+		(exclude_from_sim no)
+		(in_bom yes)
+		(on_board yes)
+		(dnp no)
+		(property "Reference" "TP5"
+			(at 162.306 29.21 90)
+			(effects
+				(font
+					(size 1.27 1.27)
+				)
+				(justify left)
+			)
+		)
+		(property "Value" "U2_VDD"
+			(at 161.2901 29.21 90)
+			(effects
+				(font
+					(size 1.27 1.27)
+				)
+				(justify left)
+				(hide yes)
+			)
+		)
+		(property "Footprint" "project footprints:TestPoint_THTPad_D2.0mm_Drill1.0mm"
+			(at 167.64 34.29 0)
+			(effects
+				(font
+					(size 1.27 1.27)
+				)
+				(hide yes)
+			)
+		)
+		(property "Datasheet" "~"
+			(at 167.64 34.29 0)
+			(effects
+				(font
+					(size 1.27 1.27)
+				)
+				(hide yes)
+			)
+		)
+		(property "Description" "test point"
+			(at 162.56 34.29 0)
+			(effects
+				(font
+					(size 1.27 1.27)
+				)
+				(hide yes)
+			)
+		)
+		(property "Subsystem" ""
+			(at 162.56 34.29 0)
+			(effects
+				(font
+					(size 1.27 1.27)
+				)
+				(hide yes)
+			)
+		)
+		(property "MPN" "(Embedded)"
+			(at 162.56 34.29 0)
+			(effects
+				(font
+					(size 1.27 1.27)
+				)
+				(hide yes)
+			)
+		)
+		(pin "1"
+		)
+		(instances
+			(project "10k-Hour-Timer-RP2040"
+				(path "/9d26b66f-2a94-42e5-8460-016e0bf95186/9c84c2c8-9981-4486-adaf-4a40ca17b6d0"
+					(reference "TP5")
+					(unit 1)
+				)

Commit message: floorplanning
Connections:
- net V_OUT: now reaches D8.2 (A), J10.1, J11.1 (Pin_1), JP13.1 (A), TP26.1
Changed lines of the file:
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@@
+		)
+	)
+	(label "V_OUT"
+		(at 228.6 106.68 0)
+		(effects
+			(font
+				(size 1.27 1.27)
+			)
+			(justify left bottom)
 		)
 	)

Commit message: floorplanning batt prot
Parts:
- added TP27: FB, project footprints:TestPoint_THTPad_D2.0mm_Drill1.0mm, symbol Connector:TestPoint
Connections:
- net DC_FB: now also TP27.1
- net DOUT: now reaches Q3.1 (G), R13.1, TP11.1, U3.3 (Dout)
- net at JP10.2 (B), R10.1: no longer C5.1
- net COUT: now reaches Q2.1 (G), R12.2, TP12.1, U3.2 (Cout)
- net Bat_V: now reaches JP10.1 (A), U3.5 (BAT)
- net Bat_V: now also C5.1
Changed lines of the file:
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@@
+	)
+	(junction
+		(at 62.23 134.62)
+		(diameter 0)
+		(color 0 0 0 0)
 	)
 	(junction
@@
 	)
 	(junction
+		(at 186.69 120.65)
+		(diameter 0)
+		(color 0 0 0 0)
+	)
+	(junction
 		(at 88.9 134.62)
 		(diameter 0)
@@
 	(junction
 		(at 162.56 34.29)
-		(diameter 0)
-		(color 0 0 0 0)
-	)
-	(junction
-		(at 52.07 134.62)
 		(diameter 0)
 		(color 0 0 0 0)
@@
 	(wire
 		(pts
-			(xy 52.07 134.62) (xy 54.61 134.62)
+			(xy 62.23 134.62) (xy 62.23 139.7)
 		)
 		(stroke
@@
 	(wire
 		(pts
-			(xy 179.07 120.65) (xy 201.93 120.65)
+			(xy 179.07 120.65) (xy 186.69 120.65)
 		)
 		(stroke
@@
 	(wire
 		(pts
-			(xy 52.07 134.62) (xy 52.07 139.7)
-		)
-		(stroke
-			(width 0)
-			(type default)
-		)
-	)
-	(wire
-		(pts
 			(xy 166.37 35.56) (xy 166.37 34.29)
 		)
@@
 	(wire
 		(pts
+			(xy 62.23 139.7) (xy 52.07 139.7)
+		)
+		(stroke
+			(width 0)
+			(type default)
+		)
+	)
+	(wire
+		(pts
 			(xy 158.75 109.22) (xy 158.75 113.03)
 		)
@@
 	(wire
 		(pts
-			(xy 50.8 134.62) (xy 52.07 134.62)
+			(xy 50.8 134.62) (xy 54.61 134.62)
 		)
 		(stroke
@@
 		(pts
 			(xy 158.75 100.33) (xy 152.4 100.33)
+		)
+		(stroke
+			(width 0)
+			(type default)
+		)
+	)
+	(wire
+		(pts
+			(xy 186.69 120.65) (xy 201.93 120.65)
 		)
 		(stroke
@@
 		)
 	)
+	(label "DOUT"
+		(at 85.09 139.7 0)
+		(effects
+			(font
+				(size 1.27 1.27)
+			)
+			(justify left bottom)
+		)
+	)
 	(label "Batt-"
 		(at 35.56 146.05 180)
@@
 		)
 	)
+	(label "COUT"
+		(at 85.09 134.62 0)
+		(effects
+			(font
+				(size 1.27 1.27)
+			)
+			(justify left bottom)
+		)
+	)
 	(label "Batt-"
 		(at 34.29 114.3 180)
@@
 			)
 			(justify right bottom)
+		)
+	)
+	(label "Bat_V"
+		(at 62.865 134.62 0)
+		(effects
+			(font
+				(size 1.27 1.27)
+			)
+			(justify left bottom)
 		)
 	)
@@
 		)
 	)
+	(symbol
+		(lib_id "Connector:TestPoint")
+		(at 186.69 120.65 180)
+		(unit 1)
+		(exclude_from_sim no)
+		(in_bom yes)
+		(on_board yes)
+		(dnp no)
+		(property "Reference" "TP27"
+			(at 188.722 125.984 0)
+			(effects
+				(font
+					(size 1.27 1.27)
+				)
+				(justify left)
+			)
+		)
+		(property "Value" "FB"
+			(at 187.9599 125.73 90)
+			(effects
+				(font
+					(size 1.27 1.27)
+				)
+				(justify left)
+				(hide yes)
+			)
+		)
+		(property "Footprint" "project footprints:TestPoint_THTPad_D2.0mm_Drill1.0mm"
+			(at 181.61 120.65 0)
+			(effects
+				(font
+					(size 1.27 1.27)
+				)
+				(hide yes)
+			)
+		)
+		(property "Datasheet" "~"
+			(at 181.61 120.65 0)
+			(effects
+				(font
+					(size 1.27 1.27)
+				)
+				(hide yes)
+			)
+		)
+		(property "Description" "test point"
+			(at 186.69 120.65 0)
+			(effects
+				(font
+					(size 1.27 1.27)
+				)
+				(hide yes)
+			)
+		)
+		(property "Subsystem" ""
+			(at 186.69 120.65 90)
+			(effects
+				(font
+					(size 1.27 1.27)
+				)
+				(hide yes)
+			)
+		)
+		(property "MPN" "(Embedded)"
+			(at 186.69 120.65 90)
+			(effects
+				(font
+					(size 1.27 1.27)
+				)
+				(hide yes)
+			)
+		)
+		(pin "1"
+		)
+		(instances
+			(project "10k-Hour-Timer-RP2040"
+				(path "/9d26b66f-2a94-42e5-8460-016e0bf95186/9c84c2c8-9981-4486-adaf-4a40ca17b6d0"
+					(reference "TP27")
+					(unit 1)
+				)
+			)
+		)
+	)
