File: kicad/05-07_MCU-LED-Driver-Displays.kicad_sch (KiCad schematic)
At the start: 65 parts, among them J5 Conn_02x05_Counter_Clockwise, J6 Conn_01x13_Pin, J7 Conn_01x03_Pin, J8 Conn_01x03_Pin, Q4 AO3400A, Q5 AO3400A, SW1 B3U-1100PM, SW2 BOOTSEL, SW3 RESET, SW4 USER_A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

Commit message: layout floorplanning
Parts:
- C12, C13, C14, C15, C16, C17, C18, C19, C20, C21, C22: footprint Capacitor_SMD:C_0805_2012Metric_Pad1.18x1.45mm_HandSolder -> Capacitor_SMD:C_0603_1608Metric_Pad1.08x0.95mm_HandSolder; Package 0805 -> 0603
Connections:
- net HSE_OUT2: now reaches C11.2, R26.2, Y1.1
- net SWCK_IN: now reaches R30.2, U6.24 (SWCLK)
- net SWDA_IN: now reaches R31.2, U6.25 (SWD)
- net XIN renamed HSE_IN
- net XOUT renamed HSE_OUT
Other:
- moved on the sheet: R30, R31
Changed lines of the file:
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@@
 	(text "Place 100Ω Rs close to pins"
 		(exclude_from_sim no)
-		(at 92.456 124.46 0)
+		(at 96.774 114.3 0)
 		(effects
 			(font
@@
 	(text "Decoupling Strategy\n- 100nF on all VDD\n- 1uF on VREG_In/Out"
 		(exclude_from_sim no)
-		(at 137.414 4.318 0)
+		(at 157.48 5.08 0)
 		(effects
 			(font
@@
 	(wire
 		(pts
-			(xy 120.65 123.19) (xy 121.92 123.19)
+			(xy 110.49 123.19) (xy 121.92 123.19)
 		)
 		(stroke
@@
 	(wire
 		(pts
-			(xy 109.22 118.11) (xy 109.22 123.19)
+			(xy 99.06 118.11) (xy 99.06 123.19)
 		)
 		(stroke
@@
 	(wire
 		(pts
-			(xy 105.41 118.11) (xy 109.22 118.11)
+			(xy 95.25 118.11) (xy 99.06 118.11)
 		)
 		(stroke
@@
 	(wire
 		(pts
-			(xy 120.65 125.73) (xy 121.92 125.73)
+			(xy 110.49 125.73) (xy 121.92 125.73)
 		)
 		(stroke
@@
 	(wire
 		(pts
-			(xy 104.14 130.81) (xy 109.22 130.81)
+			(xy 93.98 130.81) (xy 99.06 130.81)
 		)
 		(stroke
@@
 	(wire
 		(pts
-			(xy 109.22 125.73) (xy 113.03 125.73)
+			(xy 99.06 125.73) (xy 102.87 125.73)
 		)
 		(stroke
@@
 	(wire
 		(pts
-			(xy 109.22 130.81) (xy 109.22 125.73)
+			(xy 99.06 130.81) (xy 99.06 125.73)
 		)
 		(stroke
@@
 	(wire
 		(pts
-			(xy 109.22 123.19) (xy 113.03 123.19)
+			(xy 99.06 123.19) (xy 102.87 123.19)
 		)
 		(stroke
@@
 		)
 	)
-	(label "XIN"
+	(label "HSE_IN"
 		(at 69.85 125.73 180)
 		(effects
@@
 		)
 	)
-	(label "XOUT"
+	(label "HSE_OUT"
 		(at 113.03 113.03 0)
 		(effects
@@
 		)
 	)
+	(label "SWCK_IN"
+		(at 111.76 123.19 0)
+		(effects
+			(font
+				(size 1.27 1.27)
+			)
+			(justify left bottom)
+		)
+	)
 	(label "UART0_Rx"
 		(at 184.15 59.69 180)
@@
 		)
 	)
+	(label "SWDA_IN"
+		(at 111.76 125.73 0)
+		(effects
+			(font
+				(size 1.27 1.27)
+			)
+			(justify left bottom)
+		)
+	)
 	(label "ADC0"
 		(at 179.07 125.73 180)
@@
 		)
 	)
-	(label "XIN"
+	(label "HSE_IN"
 		(at 113.03 102.87 0)
 		(effects
@@
 		)
 	)
+	(label "HSE_OUT2"
+		(at 44.45 138.43 0)
+		(effects
+			(font
+				(size 1.27 1.27)
+			)
+			(justify left bottom)
+		)
+	)
 	(label "IO2"
 		(at 179.07 62.23 180)
@@
 		)
 	)
-	(label "XOUT"
+	(label "HSE_OUT"
 		(at 69.85 138.43 180)
 		(effects
@@
 	(hierarchical_label "SWD"
 		(shape input)
-		(at 104.14 130.81 180)
+		(at 93.98 130.81 180)
 		(effects
 			(font
@@
 	(hierarchical_label "SWCK"
 		(shape input)
-		(at 105.41 118.11 180)
+		(at 95.25 118.11 180)
 		(effects
 			(font
@@
 			)
 		)
-		(property "Footprint" "Capacitor_SMD:C_0805_2012Metric_Pad1.18x1.45mm_HandSolder"
+		(property "Footprint" "Capacitor_SMD:C_0603_1608Metric_Pad1.08x0.95mm_HandSolder"
 			(at 178.7652 26.67 0)
 			(effects
@@
 			)
 		)
-		(property "Package" "0805"
+		(property "Package" "0603"
 			(at 177.8 22.86 0)
 			(effects
@@
 			)
 		)
-		(property "Footprint" "Capacitor_SMD:C_0805_2012Metric_Pad1.18x1.45mm_HandSolder"
+		(property "Footprint" "Capacitor_SMD:C_0603_1608Metric_Pad1.08x0.95mm_HandSolder"
 			(at 263.8552 57.15 0)
 			(effects
@@
 			)
 		)
-		(property "Package" "0805"
+		(property "Package" "0603"
 			(at 262.89 53.34 0)
 			(effects
@@
 			)
 		)
-		(property "Footprint" "Capacitor_SMD:C_0805_2012Metric_Pad1.18x1.45mm_HandSolder"
+		(property "Footprint" "Capacitor_SMD:C_0603_1608Metric_Pad1.08x0.95mm_HandSolder"
 			(at 140.6652 26.67 0)
 			(effects
@@
 			)
 		)
-		(property "Package" "0805"
+		(property "Package" "0603"
 			(at 139.7 22.86 0)
 			(effects
@@
 			)
 		)
-		(property "Footprint" "Capacitor_SMD:C_0805_2012Metric_Pad1.18x1.45mm_HandSolder"
+		(property "Footprint" "Capacitor_SMD:C_0603_1608Metric_Pad1.08x0.95mm_HandSolder"
 			(at 190.1952 26.67 0)
 			(effects
@@
 			)
 		)
-		(property "Package" "0805"
+		(property "Package" "0603"
 			(at 189.23 22.86 0)
 			(effects
@@
 	(symbol
 		(lib_id "Device:R")
-		(at 116.84 123.19 90)
+		(at 106.68 123.19 90)
 		(unit 1)
 		(exclude_from_sim no)
@@
 		(dnp no)
 		(property "Reference" "R30"
-			(at 116.84 118.364 90)
+			(at 106.68 118.364 90)
 			(effects
 				(font
@@
 		)
 		(property "Value" "100"
-			(at 116.84 120.904 90)
+			(at 106.68 120.904 90)
 			(effects
 				(font
@@
 		)
 		(property "Footprint" "Resistor_SMD:R_0805_2012Metric_Pad1.20x1.40mm_HandSolder"
-			(at 116.84 124.968 90)
+			(at 106.68 124.968 90)
 			(effects
 				(font
@@
 		)
 		(property "Datasheet" "~"
-			(at 116.84 123.19 0)
+			(at 106.68 123.19 0)
 			(effects
 				(font
@@
 		)
 		(property "Description" "Resistor"
-			(at 116.84 123.19 0)
+			(at 106.68 123.19 0)
 			(effects
 				(font
@@
 		)
 		(property "Subsystem" "05-MCU-XTAL-FLASH"
-			(at 116.84 123.19 90)
+			(at 106.68 123.19 90)
 			(effects
 				(font
@@
 		)
 		(property "MPN" "(Generic)"
-			(at 116.84 123.19 90)
+			(at 106.68 123.19 90)
 			(effects
 				(font
@@
 		)
 		(property "Manufacturer" "(Generic)"
-			(at 116.84 123.19 90)
+			(at 106.68 123.19 90)
 			(effects
 				(font
@@
 		)
 		(property "Supplier 1" "(Generic)"
-			(at 116.84 123.19 90)
+			(at 106.68 123.19 90)
 			(effects
 				(font
@@
 		)
 		(property "Package" "0805"
-			(at 116.84 123.19 90)
+			(at 106.68 123.19 90)
 			(effects
 				(font
@@
 			)
 		)
-		(property "Footprint" "Capacitor_SMD:C_0805_2012Metric_Pad1.18x1.45mm_HandSolder"
+		(property "Footprint" "Capacitor_SMD:C_0603_1608Metric_Pad1.08x0.95mm_HandSolder"
 			(at 130.5052 26.67 0)
 			(effects
@@
 			)
 		)
-		(property "Package" "0805"
+		(property "Package" "0603"
 			(at 129.54 22.86 0)
 			(effects
@@
 			)
 		)
-		(property "Footprint" "Capacitor_SMD:C_0805_2012Metric_Pad1.18x1.45mm_HandSolder"
+		(property "Footprint" "Capacitor_SMD:C_0603_1608Metric_Pad1.08x0.95mm_HandSolder"
 			(at 167.3352 26.67 0)
 			(effects
@@
 			)
 		)
-		(property "Package" "0805"
+		(property "Package" "0603"
 			(at 166.37 22.86 0)
 			(effects
@@
 			)
 		)
-		(property "Footprint" "Capacitor_SMD:C_0805_2012Metric_Pad1.18x1.45mm_HandSolder"
+		(property "Footprint" "Capacitor_SMD:C_0603_1608Metric_Pad1.08x0.95mm_HandSolder"
 			(at 150.8252 26.67 0)
 			(effects
@@
 			)
 		)
-		(property "Package" "0805"
+		(property "Package" "0603"
 			(at 149.86 22.86 0)
 			(effects
@@
 			)
 		)
-		(property "Footprint" "Capacitor_SMD:C_0805_2012Metric_Pad1.18x1.45mm_HandSolder"
+		(property "Footprint" "Capacitor_SMD:C_0603_1608Metric_Pad1.08x0.95mm_HandSolder"
 			(at 230.8352 90.17 0)
 			(effects
@@
 			)
 		)
-		(property "Package" "0805"
+		(property "Package" "0603"
 			(at 229.87 86.36 0)
 			(effects
@@
 			)
 		)
-		(property "Footprint" "Capacitor_SMD:C_0805_2012Metric_Pad1.18x1.45mm_HandSolder"
+		(property "Footprint" "Capacitor_SMD:C_0603_1608Metric_Pad1.08x0.95mm_HandSolder"
 			(at 56.8452 81.28 0)
 			(effects
@@
 			)
 		)
-		(property "Package" "0805"
+		(property "Package" "0603"
 			(at 55.88 77.47 0)
 			(effects
@@
 			)
 		)
-		(property "Footprint" "Capacitor_SMD:C_0805_2012Metric_Pad1.18x1.45mm_HandSolder"
+		(property "Footprint" "Capacitor_SMD:C_0603_1608Metric_Pad1.08x0.95mm_HandSolder"
 			(at 163.5252 46.99 0)
 			(effects
@@
 			)
 		)
-		(property "Package" "0805"
+		(property "Package" "0603"
 			(at 162.56 43.18 0)
 			(effects
@@
 			)
 		)
-		(property "Footprint" "Capacitor_SMD:C_0805_2012Metric_Pad1.18x1.45mm_HandSolder"
+		(property "Footprint" "Capacitor_SMD:C_0603_1608Metric_Pad1.08x0.95mm_HandSolder"
 			(at 68.2752 81.28 0)
 			(effects
@@
 			)
 		)
-		(property "Package" "0805"
+		(property "Package" "0603"
 			(at 67.31 77.47 0)
 			(effects
@@
 	(symbol
 		(lib_id "Device:R")
-		(at 116.84 125.73 90)
+		(at 106.68 125.73 90)
 		(unit 1)
 		(exclude_from_sim no)
@@
 		(dnp no)
 		(property "Reference" "R31"
-			(at 116.84 128.016 90)
+			(at 106.68 128.016 90)
 			(effects
 				(font
@@
 		)
 		(property "Value" "100"
-			(at 116.84 130.556 90)
+			(at 106.68 130.556 90)
 			(effects
 				(font
@@
 		)
 		(property "Footprint" "Resistor_SMD:R_0805_2012Metric_Pad1.20x1.40mm_HandSolder"
-			(at 116.84 127.508 90)
+			(at 106.68 127.508 90)
 			(effects
 				(font
@@
 		)
 		(property "Datasheet" "~"
-			(at 116.84 125.73 0)
+			(at 106.68 125.73 0)
 			(effects
 				(font
@@
 		)
 		(property "Description" "Resistor"
-			(at 116.84 125.73 0)
+			(at 106.68 125.73 0)
 			(effects
 				(font
@@
 		)
 		(property "Subsystem" "05-MCU-XTAL-FLASH"
-			(at 116.84 125.73 90)
+			(at 106.68 125.73 90)
 			(effects
 				(font
@@
 		)
 		(property "MPN" "(Generic)"
-			(at 116.84 125.73 90)
+			(at 106.68 125.73 90)
 			(effects
 				(font
@@
 		)
 		(property "Manufacturer" "(Generic)"
-			(at 116.84 125.73 90)
+			(at 106.68 125.73 90)
 			(effects
 				(font
@@
 		)
 		(property "Supplier 1" "(Generic)"
-			(at 116.84 125.73 90)
+			(at 106.68 125.73 90)
 			(effects
 				(font
@@
 		)
 		(property "Package" "0805"
-			(at 116.84 125.73 90)
+			(at 106.68 125.73 90)
 			(effects
 				(font

Commit message: layout - 7seg display
Parts:
- added R44: 10K, Resistor_SMD:R_0805_2012Metric_Pad1.20x1.40mm_HandSolder, symbol Device:R
- R36: value 1K -> 10K
Connections:
- net BZ1: now also U6.13 (GPIO10); no longer U6.8 (GPIO6)
- net DISP_DIO: now also U6.14 (GPIO11); no longer U6.16 (GPIO13)
- net DISP_STB: now also U6.16 (GPIO13); no longer U6.14 (GPIO11)
- net at BZ2.1 (+), R32.1: now also R44.1
- net at BZ2.2 (-), JP20.1 (A): now also R44.2
- net IO10: no longer names the net of J6.7 (Pin_7)
- net IO10: no longer U6.13 (GPIO10)
Other:
- moved on the sheet: JP19, R32
Changed lines of the file:
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@@
 	)
 	(junction
+		(at 168.91 166.37)
+		(diameter 0)
+		(color 0 0 0 0)
+	)
+	(junction
 		(at 25.4 138.43)
 		(diameter 0)
@@
 	)
 	(junction
+		(at 168.91 158.75)
+		(diameter 0)
+		(color 0 0 0 0)
+	)
+	(junction
 		(at 85.09 180.34)
 		(diameter 0)
@@
 	(wire
 		(pts
+			(xy 168.91 166.37) (xy 171.45 166.37)
+		)
+		(stroke
+			(width 0)
+			(type default)
+		)
+	)
+	(wire
+		(pts
 			(xy 29.21 180.34) (xy 30.48 180.34)
 		)
@@
 	(wire
 		(pts
+			(xy 171.45 158.75) (xy 171.45 161.29)
+		)
+		(stroke
+			(width 0)
+			(type default)
+		)
+	)
+	(wire
+		(pts
 			(xy 144.78 46.99) (xy 142.24 46.99)
 		)
@@
 	(wire
 		(pts
-			(xy 154.94 166.37) (xy 171.45 166.37)
+			(xy 154.94 166.37) (xy 168.91 166.37)
 		)
 		(stroke
@@
 	(wire
 		(pts
+			(xy 168.91 158.75) (xy 171.45 158.75)
+		)
+		(stroke
+			(width 0)
+			(type default)
+		)
+	)
+	(wire
+		(pts
 			(xy 166.37 26.67) (xy 177.8 26.67)
 		)
@@
 	(wire
 		(pts
-			(xy 139.7 161.29) (xy 147.32 161.29)
+			(xy 139.7 158.75) (xy 147.32 158.75)
 		)
 		(stroke
@@
 	(wire
 		(pts
-			(xy 154.94 161.29) (xy 156.21 161.29)
+			(xy 154.94 158.75) (xy 156.21 158.75)
 		)
 		(stroke
@@
 	(wire
 		(pts
-			(xy 163.83 161.29) (xy 171.45 161.29)
+			(xy 163.83 158.75) (xy 168.91 158.75)
 		)
 		(stroke
@@
 		)
 	)
-	(label "DISP_DIO"
-		(at 184.15 90.17 180)
+	(label "STB_Out"
+		(at 95.25 180.34 180)
 		(effects
 			(font
@@
 		)
 	)
-	(label "STB_Out"
-		(at 95.25 180.34 180)
+	(label "BZ1"
+		(at 179.07 82.55 180)
 		(effects
 			(font
@@
 		)
 	)
+	(label "DISP_STB"
+		(at 184.15 90.17 180)
+		(effects
+			(font
+				(size 1.27 1.27)
+			)
+			(justify right bottom)
+		)
+	)
 	(label "UART0_Rx"
 		(at 184.15 59.69 180)
@@
 		)
 	)
-	(label "BZ1"
-		(at 184.15 72.39 180)
-		(effects
-			(font
-				(size 1.27 1.27)
-			)
-			(justify right bottom)
-		)
-	)
 	(label "IO21"
 		(at 179.07 110.49 180)
@@
 		)
 	)
-	(label "IO10"
-		(at 110.49 176.53 180)
-		(effects
-			(font
-				(size 1.27 1.27)
-			)
-			(justify right bottom)
-		)
-	)
 	(label "IO3"
 		(at 110.49 166.37 180)
@@
 		)
 	)
-	(label "DISP_STB"
-		(at 184.15 85.09 180)
-		(effects
-			(font
-				(size 1.27 1.27)
-			)
-			(justify right bottom)
-		)
-	)
 	(label "HSE_OUT2"
 		(at 44.45 138.43 0)
@@
 	)
 	(label "BZ2_P"
-		(at 139.7 161.29 0)
+		(at 139.7 158.75 0)
 		(effects
 			(font
@@
 		)
 	)
-	(label "IO10"
-		(at 179.07 82.55 180)
-		(effects
-			(font
-				(size 1.27 1.27)
-			)
-			(justify right bottom)
-		)
-	)
 	(label "QSPI_CLK"
 		(at 21.59 87.63 0)
@@
 		)
 	)
+	(label "DISP_DIO"
+		(at 184.15 85.09 180)
+		(effects
+			(font
+				(size 1.27 1.27)
+			)
+			(justify right bottom)
+		)
+	)
 	(label "IO14"
 		(at 110.49 179.07 180)
@@
 	)
 	(symbol
+		(lib_id "Device:R")
+		(at 168.91 162.56 0)
+		(unit 1)
+		(exclude_from_sim no)
+		(in_bom yes)
+		(on_board yes)
+		(dnp yes)
+		(property "Reference" "R44"
+			(at 164.338 163.068 90)
+			(effects
+				(font
+					(size 1.27 1.27)
+				)
+			)
+		)
+		(property "Value" "10K"
+			(at 166.624 162.814 90)
+			(effects
+				(font
+					(size 1.27 1.27)
+				)
+			)
+		)
+		(property "Footprint" "Resistor_SMD:R_0805_2012Metric_Pad1.20x1.40mm_HandSolder"
+			(at 167.132 162.56 90)
+			(effects
+				(font
+					(size 1.27 1.27)
+				)
+				(hide yes)
+			)
+		)
+		(property "Datasheet" "~"
+			(at 168.91 162.56 0)
+			(effects
+				(font
+					(size 1.27 1.27)
+				)
+				(hide yes)
+			)
+		)
+		(property "Description" "Resistor"
+			(at 168.91 162.56 0)
+			(effects
+				(font
+					(size 1.27 1.27)
+				)
+				(hide yes)
+			)
+		)
+		(property "Subsystem" "06-MCU-IO"
+			(at 168.91 162.56 90)
+			(effects
+				(font
+					(size 1.27 1.27)
+				)
+				(hide yes)
+			)
+		)
+		(property "MPN" "(Generic)"
+			(at 168.91 162.56 90)
+			(effects
+				(font
+					(size 1.27 1.27)
+				)
+				(hide yes)
+			)
+		)
+		(property "Package" "0805"
+			(at 168.91 162.56 90)
+			(effects
+				(font
+					(size 1.27 1.27)
+				)
+				(hide yes)
+			)
+		)
+		(property "Manufacturer" "(Generic)"
+			(at 168.91 162.56 90)
+			(effects
+				(font
+					(size 1.27 1.27)
+				)
+				(hide yes)
+			)
+		)
+		(property "Supplier 1" "(Generic)"
+			(at 168.91 162.56 90)
+			(effects
+				(font
+					(size 1.27 1.27)
+				)
+				(hide yes)
+			)
+		)
+		(pin "1"
+		)
+		(pin "2"
+		)
+		(instances
+			(project "10k-Hour-Timer-RP2040"
+				(path "/9d26b66f-2a94-42e5-8460-016e0bf95186/550d9dc0-5a0f-4821-af38-4e76d354dcfd"
+					(reference "R44")
+					(unit 1)
+				)
+			)
+		)
+	)
+	(symbol
 		(lib_id "power:GND")
 		(at 273.05 57.15 0)
@@
 	(symbol
 		(lib_id "Jumper:SolderJumper_2_Bridged")
-		(at 151.13 161.29 180)
+		(at 151.13 158.75 180)
 		(unit 1)
 		(exclude_from_sim no)
@@
 		(dnp no)
 		(property "Reference" "JP19"
-			(at 149.352 158.496 0)
+			(at 149.352 155.956 0)
 			(effects
 				(font
@@
 		)
 		(property "Value" "SolderJumper_2_Bridged"
-			(at 152.3999 158.75 90)
+			(at 152.3999 156.21 90)
 			(effects
 				(font
@@
 		)
 		(property "Footprint" "Jumper:SolderJumper-2_P1.3mm_Bridged_RoundedPad1.0x1.5mm"
-			(at 151.13 161.29 0)
+			(at 151.13 158.75 0)
 			(effects
 				(font
@@
 		)
 		(property "Datasheet" "~"
-			(at 151.13 161.29 0)
+			(at 151.13 158.75 0)
 			(effects
 				(font
@@
 		)
 		(property "Description" "Solder Jumper, 2-pole, closed/bridged"
-			(at 151.13 161.29 0)
+			(at 151.13 158.75 0)
 			(effects
 				(font
@@
 		)
 		(property "Subsystem" "06-MCU-IO"
-			(at 151.13 161.29 0)
+			(at 151.13 158.75 0)
 			(effects
 				(font
@@
 		)
 		(property "MPN" "(Embedded)"
-			(at 151.13 161.29 0)
+			(at 151.13 158.75 0)
 			(effects
 				(font
@@
 	(symbol
 		(lib_id "Device:R")
-		(at 160.02 161.29 270)
+		(at 160.02 158.75 270)
 		(unit 1)
 		(exclude_from_sim no)
@@
 		(dnp no)
 		(property "Reference" "R32"
-			(at 159.512 156.718 90)
+			(at 159.512 154.178 90)
 			(effects
 				(font
@@
 		)
 		(property "Value" "1K"
-			(at 159.766 159.004 90)
+			(at 159.766 156.464 90)
 			(effects
 				(font
@@
 		)
 		(property "Footprint" "Resistor_SMD:R_0805_2012Metric_Pad1.20x1.40mm_HandSolder"
-			(at 160.02 159.512 90)
+			(at 160.02 156.972 90)
 			(effects
 				(font
@@
 		)
 		(property "Datasheet" "~"
-			(at 160.02 161.29 0)
+			(at 160.02 158.75 0)
 			(effects
 				(font
@@
 		)
 		(property "Description" "Resistor"
-			(at 160.02 161.29 0)
+			(at 160.02 158.75 0)
 			(effects
 				(font
@@
 		)
 		(property "Subsystem" "06-MCU-IO"
-			(at 160.02 161.29 90)
+			(at 160.02 158.75 90)
 			(effects
 				(font
@@
 		)
 		(property "MPN" "(Generic)"
-			(at 160.02 161.29 90)
+			(at 160.02 158.75 90)
 			(effects
 				(font
@@
 		)
 		(property "Package" "0805"
-			(at 160.02 161.29 90)
+			(at 160.02 158.75 90)
 			(effects
 				(font
@@
 		)
 		(property "Manufacturer" "(Generic)"
-			(at 160.02 161.29 90)
+			(at 160.02 158.75 90)
 			(effects
 				(font
@@
 		)
 		(property "Supplier 1" "(Generic)"
-			(at 160.02 161.29 90)
+			(at 160.02 158.75 90)
 			(effects
 				(font
@@
 		(dnp no)
 		(property "Reference" "JP20"
-			(at 149.352 163.576 0)
+			(at 149.352 161.036 0)
 			(effects
 				(font
@@
 		(on_board yes)
 		(dnp no)
-		(fields_autoplaced yes)
 		(property "Reference" "R38"
-			(at 262.89 107.95 90)
+			(at 262.89 109.22 90)
 			(effects
 				(font
@@
 		)
 		(property "Value" "1K"
-			(at 262.89 110.49 90)
+			(at 262.89 111.76 90)
 			(effects
 				(font
@@
 			)
 		)
-		(property "Value" "1K"
+		(property "Value" "10K"
 			(at 229.362 140.97 0)
 			(effects
